File: ccd_breakout_v1.brd (EAGLE design)
At the start: 160 x 100 mm, 9 parts, among them IC2 74AS04D

Commit message: ccdDone
Parts:
- removed U$2: TCD1103, TCD1103:GLCC16
- added U$1: TCD1103_TCD1103, spectrometer_mother_board_v1:TCD1103_WQFN16X-240B
- moved R4 16.1 mm to (30.5, 19.1), turned to 90 degrees
- moved R6 13.7 mm to (34.3, 19.1), turned to 270 degrees
- moved FMMT560TC1 11.7 mm to (33.0, 25.4), turned to 0 degrees
- moved C3 9.25 mm to (20.3, 27.9)
- moved C4 9.25 mm to (24.1, 27.9)
- moved JP1 6.48 mm to (15.2, 20.3)
- moved IC2 5.39 mm to (22.9, 20.3)
- moved R5 4.27 mm to (29.2, 29.2), turned to 270 degrees
Connections:
- net GND: now also U$1.10, U$1.11, U$1.12, U$1.13, U$1.14, U$1.15, U$1.16, U$1.2, U$1.8, U$1.9; no longer U$2.10, U$2.11, U$2.12, U$2.13, U$2.14, U$2.15, U$2.16, U$2.2, U$2.8, U$2.9
- net N$10: now also U$1.5; no longer U$2.5
- net N$11: now also U$1.6; no longer U$2.6
- net N$12: now also U$1.7; no longer U$2.7
- net N$9: now also U$1.1; no longer U$2.1
- net VCC: now also U$1.3, U$1.4; no longer U$2.3, U$2.4
Routing:
- net GND: track 6.10 -> 41.4 mm
- net VCC: track 53.7 -> 35.2 mm
- net N$11: track 28.4 -> 11.9 mm
- net N$10: track 32.1 -> 15.7 mm
- net N$12: track 24.7 -> 8.87 mm
- net OS: track 20.7 -> 34.9 mm, vias 2 -> 0
- net N$8: track 3.30 -> 11.1 mm, vias 0 -> 2
- net N$9: track 4.00 -> 7.23 mm
- net N$7: track 2.60 -> 4.34 mm
- net SH: track 7.09 -> 5.60 mm
- net MCLK: track 7.09 -> 5.60 mm
- net ICG: track 7.09 -> 5.60 mm

Commit message: pcbWayCheckPassed
Changed lines of the file:
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@@
 </class>
 </classes>
-<designrules name="default">
+<designrules name="PCBWay_2layer">
 <description language="de">&lt;b&gt;EAGLE Design Rules&lt;/b&gt;
 &lt;p&gt;
@@
 <param name="mdPadVia" value="6mil"/>
 <param name="mdViaVia" value="6mil"/>
-<param name="mdSmdPad" value="6mil"/>
-<param name="mdSmdVia" value="6mil"/>
-<param name="mdSmdSmd" value="6mil"/>
-<param name="mdViaViaSameLayer" value="6mil"/>
+<param name="mdSmdPad" value="4mil"/>
+<param name="mdSmdVia" value="4mil"/>
+<param name="mdSmdSmd" value="4mil"/>
+<param name="mdViaViaSameLayer" value="8mil"/>
 <param name="mnLayersViaInSmd" value="2"/>
-<param name="mdCopperDimension" value="40mil"/>
+<param name="mdCopperDimension" value="10mil"/>
 <param name="mdDrill" value="6mil"/>
 <param name="mdSmdStop" value="0mil"/>
 <param name="msWidth" value="6mil"/>
-<param name="msDrill" value="0.35mm"/>
-<param name="msMicroVia" value="9.99mm"/>
+<param name="msDrill" value="0.3mm"/>
+<param name="msMicroVia" value="0.3mm"/>
 <param name="msBlindViaRatio" value="0.5"/>
 <param name="rvPadTop" value="0.25"/>
@@
 <param name="rvMicroViaOuter" value="0.25"/>
 <param name="rvMicroViaInner" value="0.25"/>
-<param name="rlMinPadTop" value="10mil"/>
+<param name="rlMinPadTop" value="6mil"/>
 <param name="rlMaxPadTop" value="20mil"/>
-<param name="rlMinPadInner" value="10mil"/>
+<param name="rlMinPadInner" value="6mil"/>
 <param name="rlMaxPadInner" value="20mil"/>
-<param name="rlMinPadBottom" value="10mil"/>
+<param name="rlMinPadBottom" value="6mil"/>
 <param name="rlMaxPadBottom" value="20mil"/>
-<param name="rlMinViaOuter" value="8mil"/>
+<param name="rlMinViaOuter" value="6mil"/>
 <param name="rlMaxViaOuter" value="20mil"/>
-<param name="rlMinViaInner" value="8mil"/>
+<param name="rlMinViaInner" value="6mil"/>
 <param name="rlMaxViaInner" value="20mil"/>
-<param name="rlMinMicroViaOuter" value="4mil"/>
+<param name="rlMinMicroViaOuter" value="6mil"/>
 <param name="rlMaxMicroViaOuter" value="20mil"/>
-<param name="rlMinMicroViaInner" value="4mil"/>
+<param name="rlMinMicroViaInner" value="6mil"/>
 <param name="rlMaxMicroViaInner" value="20mil"/>
 <param name="psTop" value="-1"/>
@@
 <param name="mlMinCreamFrame" value="0mil"/>
 <param name="mlMaxCreamFrame" value="0mil"/>
-<param name="mlViaStopLimit" value="0mil"/>
+<param name="mlViaStopLimit" value="0.8mm"/>
 <param name="srRoundness" value="0"/>
 <param name="srMinRoundness" value="0mil"/>
@@
 <param name="slThermalIsolate" value="10mil"/>
 <param name="slThermalsForVias" value="0"/>
-<param name="dpMaxLengthDifference" value="10mm"/>
+<param name="dpMaxLengthDifference" value="1mm"/>
 <param name="dpGapFactor" value="2.5"/>
 <param name="checkAngle" value="0"/>
