File: adc_breakout.brd (EAGLE design)
At the start: 100 x 80 mm, 14 parts, among them U1 ADS7947SRTER

Commit message: pcbWayCheckPassed
Parts:
- U1: value ADS7947SRTER -> ADS7947SRTER_ADS7947SRTER; device ADS7947SRTER:RTE16_1P7X1P7 -> spectrometer_mother_board_v1:ADS7947SRTER_RTE16_1P7X1P7
Routing:
- net GND: track 19.9 -> 9.74 mm, vias 7 -> 5
- net DVDD: track 3.55 -> 0.00 mm

Commit message: checkOK
Parts:
- SV1: value (none) -> AnalogIO
- SV2: value (none) -> DigitalIO
- U1: value ADS7947SRTER_ADS7947SRTER -> ADS7947SRTER_ADS7947SRTEREXTENDEDSOLDER; device spectrometer_mother_board_v1:ADS7947SRTER_RTE16_1P7X1P7 -> spectrometer_mother_board_v1:QFN16-EXTENDEDPADS
- turned R3 to 180 degrees
Connections:
- new net N$1: R3.2, U1.15
- net GND: now also SV1.3, SV1.4, U1.TH; no longer U1.17
- net SDO: no longer R3.2, U1.15
Routing:
- net GND: track 9.74 -> 13.6 mm, vias 5 -> 7
- net SDO: track 9.74 -> 7.35 mm
- net N$1: track 0.00 -> 2.18 mm
