File: adc_breakout.sch (EAGLE design)
At the start: 14 parts, among them U1 ADS7947SRTER

Commit message: pcbWayCheckPassed
Parts:
- U1: value ADS7947SRTER -> ADS7947SRTER_ADS7947SRTER; device ADS7947SRTER:ADS7947SRTER -> spectrometer_mother_board_v1:ADS7947SRTER_ADS7947SRTER

Commit message: checkOK
Parts:
- SV1: value (none) -> AnalogIO
- SV2: value (none) -> DigitalIO
- U1: value ADS7947SRTER_ADS7947SRTER -> ADS7947SRTER_ADS7947SRTEREXTENDEDSOLDER; device spectrometer_mother_board_v1:ADS7947SRTER_ADS7947SRTER -> spectrometer_mother_board_v1:ADS7947SRTER_ADS7947SRTEREXTENDEDSOLDER
Connections:
- new net N$1: R3.2, U1.SDO
- net GND: now also SV1.3, SV1.4
- net SDO: no longer R3.2, U1.SDO
Changed lines of the file:
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@@
 <parts>
 <part name="GND3" library="supply1" library_urn="urn:adsk.eagle:library:371" deviceset="GND" device=""/>
-<part name="SV1" library="con-lstb" library_urn="urn:adsk.eagle:library:162" deviceset="MA06-1" device="" package3d_urn="urn:adsk.eagle:package:8340/1"/>
-<part name="SV2" library="con-lstb" library_urn="urn:adsk.eagle:library:162" deviceset="MA06-1" device="" package3d_urn="urn:adsk.eagle:package:8340/1"/>
+<part name="SV1" library="con-lstb" library_urn="urn:adsk.eagle:library:162" deviceset="MA06-1" device="" package3d_urn="urn:adsk.eagle:package:8340/1" value="AnalogIO"/>
+<part name="SV2" library="con-lstb" library_urn="urn:adsk.eagle:library:162" deviceset="MA06-1" device="" package3d_urn="urn:adsk.eagle:package:8340/1" value="DigitalIO"/>
 <part name="C1" library="rcl" library_urn="urn:adsk.eagle:library:334" deviceset="C-EU" device="C0603" package3d_urn="urn:adsk.eagle:package:23616/2" value="470 pF"/>
 <part name="C2" library="rcl" library_urn="urn:adsk.eagle:library:334" deviceset="C-EU" device="C0603" package3d_urn="urn:adsk.eagle:package:23616/2" value="470 pF"/>
@@
 <part name="C5" library="rcl" library_urn="urn:adsk.eagle:library:334" deviceset="C-EU" device="C0603" package3d_urn="urn:adsk.eagle:package:23616/2" value="1 uF"/>
 <part name="C6" library="rcl" library_urn="urn:adsk.eagle:library:334" deviceset="C-EU" device="C0603" package3d_urn="urn:adsk.eagle:package:23616/2" value="1 uF"/>
-<part name="U1" library="spectrometer_mother_board_v1" deviceset="ADS7947SRTER_ADS7947SRTER" device=""/>
+<part name="U1" library="spectrometer_mother_board_v1" deviceset="ADS7947SRTER_ADS7947SRTER" device="EXTENDEDSOLDER" value="ADS7947SRTER_ADS7947SRTEREXTENDEDSOLDER"/>
 </parts>
 <sheets>
@@
 </instance>
 <instance part="SV2" gate="1" x="142.24" y="45.72" smashed="yes" rot="R180">
-<attribute name="VALUE" x="143.51" y="58.42" size="1.778" layer="96" rot="R180"/>
+<attribute name="VALUE" x="144.78" y="38.1" size="1.778" layer="96" rot="R180"/>
 <attribute name="NAME" x="138.43" y="57.658" size="1.778" layer="95" rot="MR180" align="top-left"/>
 </instance>
@@
 <wire x1="76.2" y1="96.52" x2="76.2" y2="93.98" width="0.1524" layer="91"/>
 </segment>
+<segment>
+<pinref part="SV1" gate="1" pin="4"/>
+<wire x1="-20.32" y1="48.26" x2="-17.78" y2="48.26" width="0.1524" layer="91"/>
+<pinref part="SV1" gate="1" pin="3"/>
+<wire x1="-17.78" y1="48.26" x2="-17.78" y2="45.72" width="0.1524" layer="91"/>
+<wire x1="-17.78" y1="45.72" x2="-20.32" y2="45.72" width="0.1524" layer="91"/>
+<label x="-17.78" y="48.26" size="1.778" layer="95"/>
+</segment>
 </net>
 <net name="CHSEL" class="0">
@@
 </net>
 <net name="SDO" class="0">
-<segment>
-<wire x1="78.74" y1="50.8" x2="106.68" y2="50.8" width="0.1524" layer="91"/>
-<pinref part="R3" gate="G$1" pin="2"/>
-<pinref part="U1" gate="A" pin="SDO"/>
-</segment>
 <segment>
 <pinref part="R3" gate="G$1" pin="1"/>
@@
 </segment>
 </net>
+<net name="N$1" class="0">
+<segment>
+<pinref part="U1" gate="A" pin="SDO"/>
+<pinref part="R3" gate="G$1" pin="2"/>
+<wire x1="78.74" y1="50.8" x2="106.68" y2="50.8" width="0.1524" layer="91"/>
+</segment>
+</net>
